File: MCU_circuits/MCU_circuits.kicad_sch (KiCad schematic)
At the start: 67 parts, among them J1 COLOR_program, J11 UI_program, J12 power_ISP, J13 TEENSY_4.1_to_UI, J2 TEENSY_4.1_to_COLOR, J3 COLOR_to_PC, J4 POWER, J5 power_program, J6 TEENSY_4.1_to_MD, J7 USB_C_Receptacle_USB2.0_16P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

Commit message: 急いでコピペしてわかりずらいコネクター名を変更
Parts:
- J13: value TEENSY_4.1_to_UI -> connect
- J2: value TEENSY_4.1_to_COLOR -> connect
- J6: value TEENSY_4.1_to_MD -> connect
Changed lines of the file:
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@@
 			)
 		)
-		(property "Value" "TEENSY_4.1_to_MD"
+		(property "Value" "connect"
 			(at 246.38 299.7199 0)
 			(effects
@@
 			)
 		)
-		(property "Value" "TEENSY_4.1_to_COLOR"
+		(property "Value" "connect"
 			(at 49.53 255.2699 0)
 			(effects
@@
 			)
 		)
-		(property "Value" "TEENSY_4.1_to_UI"
+		(property "Value" "connect"
 			(at 433.07 231.1399 0)
 			(effects
