File: Rocket_CDR_1/Rocket_CDR_1.kicad_sch (KiCad schematic)
At the start: 52 parts, among them J1 BATT, J2 BATT, Q1 VTT9812FH, SW1 SW_SPST, SW2 SW_Push, SW3 SW_Push, U1 BD50FC0FP

Commit message: ダイオードの追加
Parts:
- added D8: D, symbol Device:D
Connections:
- net +5V: now also D8.2 (A)
- net batt: now also D8.1 (K)
Other:
- moved on the sheet: J2
